Commit message: introduced ros2_control and tested moving in gazebo simulation

File: src/vision_bot/description/robot.urdf.xacro (robot description, xacro)
@@ -1,4 +1,5 @@
 <?xml version="1.0"?>
 <robot name="robot" xmlns:xacro="http://www.ros.org/wiki/xacro">
-    <xacro:include filename="robot_core.xacro"/>
+    <xacro:include filename="robot_core.xacro" />
+    <xacro:include filename="ros2_control.xacro" />
 </robot>

File: src/vision_bot/description/robot_core.xacro (robot description, xacro)
@@ -22,5 +22,5 @@
     <link name="chassis">
         <visual>
-            <origin xyz="0 0 0.075"/>
+            <origin xyz="0 0 0.1"/>
             <geometry>
                 <box size="0.4 0.3 0.15"/>
@@ -29,5 +29,5 @@
         </visual>
         <collision>
-            <origin xyz="0 0 0.075"/>
+            <origin xyz="0 0 0.1"/>
             <geometry>
                 <box size="0.4 0.3 0.15"/>
@@ -43,5 +43,5 @@
         <parent link="chassis"/>
         <child link="rear_left_wheel"/>
-        <origin xyz="-0.1 0.175 0" rpy="-${pi/2} 0 0"/>
+        <origin xyz="-0.1 0.175 0.05" rpy="-${pi/2} 0 0"/>
         <axis xyz="0 0 1"/>
     </joint>
@@ -67,5 +67,5 @@
         <parent link="chassis"/>
         <child link="rear_right_wheel"/>
-        <origin xyz="-0.1 -0.175 0" rpy="${pi/2} 0 0"/>
+        <origin xyz="-0.1 -0.175 0.05" rpy="${pi/2} 0 0"/>
         <axis xyz="0 0 -1"/>
     </joint>
@@ -91,5 +91,5 @@
         <parent link="chassis"/>
         <child link="front_left_wheel"/>
-        <origin xyz="0.1 0.175 0" rpy="-${pi/2} 0 0"/>
+        <origin xyz="0.1 0.175 0.05" rpy="-${pi/2} 0 0"/>
         <axis xyz="0 0 1"/>
     </joint>
@@ -115,6 +115,6 @@
         <parent link="chassis"/>
         <child link="front_right_wheel"/>
-        <origin xyz="0.1 -0.175 0" rpy="-${pi/2} 0 0"/>
-        <axis xyz="0 0 1"/>
+        <origin xyz="0.1 -0.175 0.05" rpy="${pi/2} 0 0"/>
+        <axis xyz="0 0 -1"/>
     </joint>
     <link name="front_right_wheel">
