Commit message: changed xacro configuration & added camera sensor in simulation

File: src/vision_bot/description/robot_core.xacro (robot description, xacro)
@@ -1,5 +1,5 @@
 <?xml version="1.0"?>
 <robot name="robot" xmlns:xacro="http://www.ros.org/wiki/xacro">
-    <xacro:include filename="inertia_macros.xacro"/>
+    <!-- COLORS -->
     <material name="white">
         <color rgba="1 1 1 1"/>
@@ -14,124 +14,6 @@
     <link name="base_link">
     </link>
-    <!-- CHASSIS LINK -->
-    <joint name="chassis_joint" type="fixed">
-        <parent link="base_link"/>
-        <child link="chassis"/>
-        <origin xyz="0 0 0"/>
-    </joint>
-    <link name="chassis">
-        <visual>
-            <origin xyz="0 0 0.1"/>
-            <geometry>
-                <box size="0.4 0.3 0.15"/>
-            </geometry>
-            <material name="orange"/>
-        </visual>
-        <collision>
-            <origin xyz="0 0 0.1"/>
-            <geometry>
-                <box size="0.4 0.3 0.15"/>
-            </geometry>
-            <material name="orange"/>
-        </collision>
-        <xacro:inertial_box mass="0.5" x="0.4" y="0.3" z="0.15">
-            <origin xyz="0 0 0.075" rpy="0 0 0"/>
-        </xacro:inertial_box>
-    </link>
-    <!-- LEFT REAR WHEEL LINK -->
-    <joint name="rear_left_wheel_joint" type="continuous">
-        <parent link="chassis"/>
-        <child link="rear_left_wheel"/>
-        <origin xyz="-0.1 0.175 0.05" rpy="-${pi/2} 0 0"/>
-        <axis xyz="0 0 1"/>
-    </joint>
-    <link name="rear_left_wheel">
-        <visual>
-            <geometry>
-                <cylinder radius="0.05" length="0.05"/>
-            </geometry>
-            <material name="black"/>
-        </visual>
-        <collision>
-            <geometry>
-                <cylinder radius="0.05" length="0.05"/>
-            </geometry>
-            <material name="black"/>
-        </collision>
-        <xacro:inertial_cylinder mass="0.1" length="0.05" radius="0.05">
-            <origin xyz="0 0 0" rpy="0 0 0"/>
-        </xacro:inertial_cylinder>
-    </link>
-    <!-- RIGHT REAR WHEEL LINK -->
-    <joint name="rear_right_wheel_joint" type="continuous">
-        <parent link="chassis"/>
-        <child link="rear_right_wheel"/>
-        <origin xyz="-0.1 -0.175 0.05" rpy="${pi/2} 0 0"/>
-        <axis xyz="0 0 -1"/>
-    </joint>
-    <link name="rear_right_wheel">
-        <visual>
-            <geometry>
-                <cylinder radius="0.05" length="0.05"/>
-            </geometry>
-            <material name="black"/>
-        </visual>
-        <collision>
-            <geometry>
-                <cylinder radius="0.05" length="0.05"/>
-            </geometry>
-            <material name="black"/>
-        </collision>
-        <xacro:inertial_cylinder mass="0.1" length="0.05" radius="0.05">
-            <origin xyz="0 0 0" rpy="0 0 0"/>
-        </xacro:inertial_cylinder>
-    </link>
-    <!-- LEFT FRONT WHEEL LINK -->
-    <joint name="front_left_wheel_joint" type="continuous">
-        <parent link="chassis"/>
-        <child link="front_left_wheel"/>
-        <origin xyz="0.1 0.175 0.05" rpy="-${pi/2} 0 0"/>
-        <axis xyz="0 0 1"/>
-    </joint>
-    <link name="front_left_wheel">
-        <visual>
-            <geometry>
-                <cylinder radius="0.05" length="0.05"/>
-            </geometry>
-            <material name="black"/>
-        </visual>
-        <collision>
-            <geometry>
-                <cylinder radius="0.05" length="0.05"/>
-            </geometry>
-            <material name="black"/>
-        </collision>
-        <xacro:inertial_cylinder mass="0.1" length="0.05" radius="0.05">
-            <origin xyz="0 0 0" rpy="0 0 0"/>
-        </xacro:inertial_cylinder>
-    </link>
-    <!-- RIGHT FRONT WHEEL LINK -->
-    <joint name="front_right_wheel_joint" type="continuous">
-        <parent link="chassis"/>
-        <child link="front_right_wheel"/>
-        <origin xyz="0.1 -0.175 0.05" rpy="${pi/2} 0 0"/>
-        <axis xyz="0 0 -1"/>
-    </joint>
-    <link name="front_right_wheel">
-        <visual>
-            <geometry>
-                <cylinder radius="0.05" length="0.05"/>
-            </geometry>
-            <material name="black"/>
-        </visual>
-        <collision>
-            <geometry>
-                <cylinder radius="0.05" length="0.05"/>
-            </geometry>
-            <material name="black"/>
-        </collision>
-        <xacro:inertial_cylinder mass="0.1" length="0.05" radius="0.05">
-            <origin xyz="0 0 0" rpy="0 0 0"/>
-        </xacro:inertial_cylinder>
-    </link>
+    <xacro:include filename="components/chassis.xacro" />
+    <xacro:include filename="components/wheels.xacro" />
+    <xacro:include filename="components/camera.xacro" />
 </robot>
