Commit message: added front ultrasonic sensor in simulation environment

File: src/vision_bot/description/components/camera.xacro (robot description, xacro)
@@ -5,5 +5,4 @@
     <xacro:property name="camera_neck_width" value="0.01"/>
     <xacro:property name="camera_neck_height" value="0.015"/>
-    <xacro:property name="camera_neck_mass" value="0.01"/>
     <xacro:property name="camera_length" value="0.01" />
     <xacro:property name="camera_width" value="0.015"/>
@@ -51,5 +50,4 @@
             <update_rate>30</update_rate>
             <topic>camera/image_raw</topic>
-            <gz_frame_id>camera_rgb_frame</gz_frame_id>
             <camera>
                 <camera_info_topic>camera/camera_info</camera_info_topic>

File: src/vision_bot/description/robot_core.xacro (robot description, xacro)
@@ -8,4 +8,7 @@
         <color rgba="1 0.3 0.1 1"/>
     </material>
+    <material name="blue">
+        <color rgba="0 0.2588 0.51 1"/>
+    </material>
     <material name="black">
         <color rgba="0 0 0 1"/>
@@ -14,6 +17,8 @@
     <link name="base_link">
     </link>
+    <!-- COMPONENTS -->
     <xacro:include filename="components/chassis.xacro" />
     <xacro:include filename="components/wheels.xacro" />
     <xacro:include filename="components/camera.xacro" />
+    <xacro:include filename="components/uss.xacro" />
 </robot>

File: src/vision_bot/description/ros2_control.xacro (robot description, xacro)
@@ -30,4 +30,7 @@
             <parameters>$(find vision_bot)/config/controllers.yaml</parameters>
         </plugin>
+        <plugin name="gz::sim::systems::Sensors"
+                filename="gz-sim-sensors-system">
+        </plugin>
     </gazebo>
 </robot>

Commit message: add front left and right uss

File: src/vision_bot/description/components/camera.xacro (robot description, xacro)
@@ -11,5 +11,5 @@
     <xacro:property name="chassis_length" value="0.2" />
     <xacro:property name="chassis_height" value="0.05"/>
-    <xacro:property name="camera_neck_offset_x" value="${chassis_length - 0.03}" />
+    <xacro:property name="camera_neck_offset_x" value="${chassis_length - 0.005}" />
     <xacro:property name="camera_neck_offset_z" value="${chassis_height + (camera_neck_height / 2)}" />
     <xacro:property name="camera_offset_z" value="${(camera_neck_height/2) + (camera_height / 2)}" />
@@ -30,5 +30,5 @@
         <parent link="camera_neck_link"/>
         <child link="camera_link"/>
-        <origin xyz="0 0 ${camera_offset_z}" rpy="0 0 0"/>
+        <origin xyz="0.002 0 ${camera_offset_z}" rpy="0 0.15 0"/>
     </joint>
     <link name="camera_link">

File: src/vision_bot/description/components/uss.xacro (robot description, xacro)
@@ -7,12 +7,40 @@
     <xacro:property name="uss_width" value="0.04"/>
     <xacro:property name="uss_height" value="0.015"/>
-    <xacro:property name="uss_offset_x" value="${chassis_length + (uss_height / 2)}" />
+    <xacro:property name="uss_offset_x" value="${chassis_length + (uss_height / 2) + 0.01}" />
     <xacro:property name="uss_offset_z" value="${chassis_offset_z}"/>
+    <xacro:property name="uss_side_offset_y" value="0.043" />
+    <xacro:property name="uss_side_angle" value="0.45" />
     <joint name="front_uss_joint" type="fixed">
         <parent link="chassis"/>
         <child link="front_uss_link"/>
-        <origin xyz="${uss_offset_x} 0 ${uss_offset_z}" rpy="0 0 0"/>
+        <origin xyz="${uss_offset_x + 0.01} 0 ${uss_offset_z}" rpy="0 0 0"/>
     </joint>
     <link name="front_uss_link">
+        <visual>
+            <geometry>
+                <box size="${uss_length} ${uss_width} ${uss_height}"/>
+            </geometry>
+            <material name="blue"/>
+        </visual>
+    </link>
+    <joint name="front_left_uss_joint" type="fixed">
+        <parent link="chassis"/>
+        <child link="front_left_uss_link"/>
+        <origin xyz="${uss_offset_x} ${uss_side_offset_y} ${uss_offset_z}" rpy="0 0 ${uss_side_angle}"/>
+    </joint>
+    <link name="front_left_uss_link">
+        <visual>
+            <geometry>
+                <box size="${uss_length} ${uss_width} ${uss_height}"/>
+            </geometry>
+            <material name="blue"/>
+        </visual>
+    </link>
+    <joint name="front_right_uss_joint" type="fixed">
+        <parent link="chassis"/>
+        <child link="front_right_uss_link"/>
+        <origin xyz="${uss_offset_x} -${uss_side_offset_y} ${uss_offset_z}" rpy="0 0 -${uss_side_angle}"/>
+    </joint>
+    <link name="front_right_uss_link">
         <visual>
             <geometry>
