Commit message: world added, robot model changed

File: src/vision_bot/description/components/camera.xacro (robot description, xacro)
@@ -2,15 +2,12 @@
 <robot name="robot" xmlns:xacro="http://www.ros.org/wiki/xacro">
     <xacro:include filename="inertia_macros.xacro" />
-    <xacro:property name="camera_neck_length" value="0.01" />
+    <xacro:property name="camera_neck_length" value="0.001" />
     <xacro:property name="camera_neck_width" value="0.01"/>
-    <xacro:property name="camera_neck_height" value="0.015"/>
-    <xacro:property name="camera_length" value="0.01" />
-    <xacro:property name="camera_width" value="0.015"/>
+    <xacro:property name="camera_neck_height" value="0.01"/>
     <xacro:property name="camera_height" value="0.01"/>
-    <xacro:property name="camera_mass" value="0.01"/>
-    <xacro:property name="chassis_length" value="0.2" />
-    <xacro:property name="chassis_height" value="0.05"/>
-    <xacro:property name="camera_neck_offset_x" value="${chassis_length - 0.005}" />
-    <xacro:property name="camera_neck_offset_z" value="${chassis_height + (camera_neck_height / 2)}" />
+    <xacro:property name="chassis_length" value="0.17" />
+    <xacro:property name="chassis_height" value="0.035"/>
+    <xacro:property name="camera_neck_offset_x" value="${(chassis_length/3) + 0.01}" />
+    <xacro:property name="camera_neck_offset_z" value="${chassis_height + (camera_neck_height / 2) - 0.015}" />
     <xacro:property name="camera_offset_z" value="${(camera_neck_height/2) + (camera_height / 2)}" />
     <joint name="camera_neck_joint" type="fixed">
@@ -24,18 +21,29 @@
                 <box size="${camera_neck_length} ${camera_neck_width} ${camera_neck_height}"/>
             </geometry>
-            <material name="orange"/>
+            <material name="white"/>
         </visual>
+        <collision>
+            <origin xyz="0 0 0" />
+            <geometry>
+                <box size="${camera_neck_length} ${camera_neck_width} ${camera_neck_height}"/>
+            </geometry>
+            <material name="white"/>
+        </collision>
+        <xacro:inertial_box mass="0.1" x="${camera_neck_length}" y="${camera_neck_width}" z="${camera_neck_height}">
+            <origin xyz="0 0 0" rpy="0 0 0"/>
+        </xacro:inertial_box>
     </link>
     <joint name="camera_joint" type="fixed">
         <parent link="camera_neck_link"/>
         <child link="camera_link"/>
-        <origin xyz="0.002 0 ${camera_offset_z}" rpy="0 0.15 0"/>
+        <origin xyz="0.0075 0 ${camera_offset_z}" rpy="0 ${pi/2} 0"/>
     </joint>
     <link name="camera_link">
         <visual>
+            <origin xyz="0 0 0"/>
             <geometry>
-                <box size="${camera_length} ${camera_width} ${camera_height}"/>
+                <mesh filename="package://vision_bot/description/meshes/rpi_camera_link.stl"/>
             </geometry>
-            <material name="white"/>
+            <material name="green" />
         </visual>
     </link>

File: src/vision_bot/description/components/chassis.xacro (robot description, xacro)
@@ -2,12 +2,12 @@
 <robot name="robot" xmlns:xacro="http://www.ros.org/wiki/xacro">
     <xacro:include filename="inertia_macros.xacro" />
-    <xacro:property name="chassis_length" value="0.2" />
-    <xacro:property name="chassis_width" value="0.135"/>
-    <xacro:property name="chassis_height" value="0.05"/>
+    <xacro:property name="chassis_length" value="0.17" />
+    <xacro:property name="chassis_width" value="0.1"/>
+    <xacro:property name="chassis_height" value="0.035"/>
     <xacro:property name="chassis_mass" value="1.5"/>
-    <xacro:property name="chassis_offset_z" value="0.018"/>
+    <xacro:property name="chassis_offset_z" value="0.037"/>
     <xacro:property name="cpu_length" value="0.085" />
-    <xacro:property name="cpu_width" value="0.056"/>
-    <xacro:property name="cpu_height" value="0.0015"/>
+    <xacro:property name="cpu_width" value="0.003"/>
+    <xacro:property name="cpu_height" value="0.02"/>
     <xacro:property name="cpu_mass" value="0.1"/>
     <!-- CHASSIS LINK -->
@@ -19,12 +19,12 @@
     <link name="chassis">
         <visual>
-            <origin xyz="${chassis_length/2} 0 ${chassis_height/2}" />
+            <origin xyz="0 0 0"/>
             <geometry>
-                <box size="${chassis_length} ${chassis_width} ${chassis_height}" />
+                <mesh filename="package://vision_bot/description/meshes/robot_base_link.stl"/>
             </geometry>
             <material name="black" />
         </visual>
         <collision>
-            <origin xyz="${chassis_length/2} 0 ${chassis_height/2}" />
+            <origin xyz="0 0 0" />
             <geometry>
                 <box size="${chassis_length} ${chassis_width} ${chassis_height}" />
@@ -33,18 +33,20 @@
         </collision>
         <xacro:inertial_box mass="${chassis_mass}" x="${chassis_length}" y="${chassis_width}" z="${chassis_height}">
-            <origin xyz="${chassis_length/2} 0 ${chassis_height/2}" rpy="0 0 0"/>
+            <origin xyz="0 0 0" rpy="0 0 0"/>
         </xacro:inertial_box>
     </link>
+    <!-- CPU LINK -->
     <joint name="cpu_joint" type="fixed">
         <parent link="chassis" />
         <child link="cpu_link" />
-        <origin xyz="${chassis_length / 2} 0 ${chassis_height + (cpu_height / 2)}" rpy="0 0 0"/>
+        <origin xyz="0 0 ${(cpu_height / 2) - 0.005}" rpy="${pi/2} 0 0"/>
     </joint>
     <link name="cpu_link">
         <visual>
+            <origin xyz="0 0 0"/>
             <geometry>
-                <box size="${cpu_length} ${cpu_width} ${cpu_height}"/>
+                <mesh filename="package://vision_bot/description/meshes/rpi5_link.stl"/>
             </geometry>
-            <material name="orange" />
+            <material name="green" />
         </visual>
         <collision>
@@ -52,5 +54,5 @@
                 <box size="${cpu_length} ${cpu_width} ${cpu_height}"/>
             </geometry>
-            <material name="orange" />
+            <material name="green" />
         </collision>
         <xacro:inertial_box mass="${cpu_mass}" x="${cpu_length}" y="${cpu_width}" z="${cpu_height}">

File: src/vision_bot/description/components/inertia_macros.xacro (robot description, xacro)
@@ -1,6 +1,4 @@
 <?xml version="1.0"?>
 <robot xmlns:xacro="http://www.ros.org/wiki/xacro">
-    <!-- Specify some standard inertial calculations https://en.wikipedia.org/wiki/List_of_moments_of_inertia -->
-    <!-- These make use of xacro's mathematical functionality -->
     <xacro:macro name="inertial_sphere" params="mass radius *origin">
         <inertial>
@@ -30,3 +28,15 @@
         </inertial>
     </xacro:macro>
+    <xacro:macro name="inertial_lidar">
+        <inertial>
+        <origin xyz="-0.011945780406062 -0.000381929217680526 -0.0170649378129477" rpy="0 0 0" />
+        <mass value="0.073084435549317" />
+        <inertia ixx="1.96074931730795E-05"
+                 ixy="-3.62091076640009E-07"
+                 ixz="4.28230084046735E-07"
+                 iyy="2.40983835136327E-05"
+                 iyz="1.50180909250652E-08"
+                 izz="4.14184164228595E-05" />
+    </inertial>
+    </xacro:macro>
 </robot>

File: src/vision_bot/description/components/uss.xacro (robot description, xacro)
@@ -10,5 +10,5 @@
     <xacro:property name="uss_offset_z" value="${chassis_offset_z}"/>
     <xacro:property name="uss_side_offset_y" value="0.043" />
-    <xacro:property name="uss_side_angle" value="0.45" />
+    <xacro:property name="uss_side_angle" value="0.785" />
     <joint name="front_uss_joint" type="fixed">
         <parent link="chassis"/>
@@ -74,3 +74,51 @@
         </sensor>
     </gazebo>
+    <gazebo reference="front_left_uss_link">
+        <sensor name="sonar_front_left" type="gpu_lidar">
+            <topic>robot/sonar_front_left</topic>
+            <pose> 0 0 0 0 0 0 </pose>
+            <visualize>false</visualize>
+            <update_rate>10</update_rate>
+            <lidar>
+                <scan>
+                    <horizontal>
+                        <samples>10</samples>
+                        <min_angle>-0.01</min_angle>
+                        <max_angle>0.01</max_angle>
+                    </horizontal>
+                </scan>
+                <range>
+                    <min>0.3</min>
+                    <max>12</max>
+                </range>
+            </lidar>
+            <always_on>1</always_on>
+            <visualize>true</visualize>
+            <gz_frame_id>laser_frame</gz_frame_id>
+        </sensor>
+    </gazebo>
+    <gazebo reference="front_right_uss_link">
+        <sensor name="sonar_front_right" type="gpu_lidar">
+            <topic>robot/sonar_front_right</topic>
+            <pose> 0 0 0 0 0 0 </pose>
+            <visualize>false</visualize>
+            <update_rate>10</update_rate>
+            <lidar>
+                <scan>
+                    <horizontal>
+                        <samples>10</samples>
+                        <min_angle>-0.01</min_angle>
+                        <max_angle>0.01</max_angle>
+                    </horizontal>
+                </scan>
+                <range>
+                    <min>0.3</min>
+                    <max>12</max>
+                </range>
+            </lidar>
+            <always_on>1</always_on>
+            <visualize>true</visualize>
+            <gz_frame_id>laser_frame</gz_frame_id>
+        </sensor>
+    </gazebo>
 </robot>

File: src/vision_bot/description/components/wheels.xacro (robot description, xacro)
@@ -2,13 +2,13 @@
 <robot name="robot" xmlns:xacro="http://www.ros.org/wiki/xacro">
     <xacro:include filename="inertia_macros.xacro" />
-    <xacro:property name="wheel_radius" value="0.034"/>
-    <xacro:property name="wheel_length" value="0.02"/>
+    <xacro:property name="wheel_radius" value="0.033"/>
+    <xacro:property name="wheel_length" value="0.022"/>
     <xacro:property name="wheel_mass" value="0.1"/>
-    <xacro:property name="chassis_length" value="0.2" />
-    <xacro:property name="chassis_width" value="0.135"/>
-    <xacro:property name="chassis_offset_z" value="0.018"/>
-    <xacro:property name="front_wheel_offset_x" value="${chassis_length - wheel_radius}"/>
-    <xacro:property name="rear_wheel_offset_x" value="${wheel_radius}"/>
-    <xacro:property name="wheel_offset_y" value="${(chassis_width/2) + (wheel_length/2)}"/>
+    <xacro:property name="chassis_length" value="0.165" />
+    <xacro:property name="chassis_width" value="0.1"/>
+    <xacro:property name="chassis_offset_z" value="0.037"/>
+    <xacro:property name="front_wheel_offset_x" value="${(chassis_length/2) - (wheel_radius/2)}"/>
+    <xacro:property name="rear_wheel_offset_x" value="${-((chassis_length/2) - (wheel_radius/2))}"/>
+    <xacro:property name="wheel_offset_y" value="${(chassis_width/2) + (wheel_length/2) + 0.015}"/>
     <xacro:property name="wheel_offset_z" value="${wheel_radius - chassis_offset_z}"/>
     <!-- LEFT REAR WHEEL LINK -->
@@ -20,10 +20,4 @@
     </joint>
     <link name="rear_left_wheel">
-        <visual>
-            <geometry>
-                <cylinder radius="${wheel_radius}" length="${wheel_length}"/>
-            </geometry>
-            <material name="orange"/>
-        </visual>
         <collision>
             <geometry>
@@ -44,10 +38,4 @@
     </joint>
     <link name="rear_right_wheel">
-        <visual>
-            <geometry>
-                <cylinder radius="${wheel_radius}" length="${wheel_length}"/>
-            </geometry>
-            <material name="orange"/>
-        </visual>
         <collision>
             <geometry>
@@ -68,10 +56,4 @@
     </joint>
     <link name="front_left_wheel">
-        <visual>
-            <geometry>
-                <cylinder radius="${wheel_radius}" length="${wheel_length}"/>
-            </geometry>
-            <material name="orange"/>
-        </visual>
         <collision>
             <geometry>
@@ -92,10 +74,4 @@
     </joint>
     <link name="front_right_wheel">
-        <visual>
-            <geometry>
-                <cylinder radius="${wheel_radius}" length="${wheel_length}"/>
-            </geometry>
-            <material name="orange"/>
-        </visual>
         <collision>
             <geometry>

File: src/vision_bot/description/robot.urdf.xacro (robot description, xacro)
@@ -2,4 +2,6 @@
 <robot name="robot" xmlns:xacro="http://www.ros.org/wiki/xacro">
     <xacro:include filename="robot_core.xacro" />
-    <xacro:include filename="ros2_control.xacro" />
+    <!-- <xacro:include filename="ros2_control.xacro" /> -->
+    <xacro:include filename="robot_control.xacro" />
+    <xacro:include filename="robot_gazebo.xacro" />
 </robot>

File: src/vision_bot/description/robot_core.xacro (robot description, xacro)
@@ -3,22 +3,21 @@
     <!-- COLORS -->
     <material name="white">
-        <color rgba="1 1 1 1"/>
+        <color rgba="0.8 0.8 0.8 1"/>
     </material>
     <material name="orange">
         <color rgba="1 0.3 0.1 1"/>
     </material>
-    <material name="blue">
-        <color rgba="0 0.2588 0.51 1"/>
+    <material name="black">
+        <color rgba="0.1 0.1 0.1 1"/>
     </material>
-    <material name="black">
-        <color rgba="0 0 0 1"/>
+    <material name="green">
+        <color rgba="0.32 0.545 0.298 1"/>
     </material>
     <!-- BASE LINK -->
-    <link name="base_link">
-    </link>
+    <link name="base_link" />
     <!-- COMPONENTS -->
     <xacro:include filename="components/chassis.xacro" />
     <xacro:include filename="components/wheels.xacro" />
     <xacro:include filename="components/camera.xacro" />
-    <xacro:include filename="components/uss.xacro" />
+    <xacro:include filename="components/lidar.xacro" />
 </robot>
