Commit message: fix gazebo sim

File: src/visionbot_description/description/components/camera.xacro (robot description, xacro)
@@ -45,5 +45,5 @@
       <origin xyz="0 0 0" />
       <geometry>
-        <mesh filename="package://visionbot_description/meshes/rpi_camera_link.stl" />
+        <mesh filename="package://visionbot_description/description/meshes/rpi_camera_link.stl" />
       </geometry>
       <material name="green" />

File: src/visionbot_description/description/components/chassis.xacro (robot description, xacro)
@@ -21,5 +21,5 @@
       <origin xyz="0 0 0" />
       <geometry>
-        <mesh filename="package://visionbot_description/meshes/robot_base_link.stl" />
+        <mesh filename="package://visionbot_description/description/meshes/robot_base_link.stl" />
       </geometry>
       <material name="black" />
@@ -47,5 +47,5 @@
       <origin xyz="0 0 0" />
       <geometry>
-        <mesh filename="package://visionbot_description/meshes/rpi5_link.stl" />
+        <mesh filename="package://visionbot_description/description/meshes/rpi5_link.stl" />
       </geometry>
       <material name="green" />

File: src/visionbot_description/description/components/lidar.xacro (robot description, xacro)
@@ -8,5 +8,5 @@
       <origin xyz="0 0 0" rpy="0 0 0" />
       <geometry>
-        <mesh filename="package://visionbot_description/meshes/laser_link.stl" />
+        <mesh filename="package://visionbot_description/description/meshes/laser_link.stl" />
       </geometry>
       <material name="black" />
@@ -15,5 +15,5 @@
       <origin xyz="0 0 0" rpy="0 0 0" />
       <geometry>
-        <mesh filename="package://visionbot_description/meshes/laser_link.stl" />
+        <mesh filename="package://visionbot_description/description/meshes/laser_link.stl" />
       </geometry>
     </collision>

File: src/visionbot_description/description/robot_gazebo.xacro (robot description, xacro)
@@ -69,5 +69,5 @@
   <gazebo>
     <plugin filename="gz_ros2_control-system" name="gz_ros2_control::GazeboSimROS2ControlPlugin">
-      <parameters>$(find visionbot_description)/config/controllers.yaml</parameters>
+      <parameters>$(find visionbot_launch)/config/controllers.yaml</parameters>
     </plugin>
     <plugin filename="gz-sim-sensors-system" name="gz::sim::systems::Sensors">

Commit message: added planning and navigation

File: src/visionbot_description/description/components/camera.xacro (robot description, xacro)
@@ -49,4 +49,9 @@
       <material name="green" />
     </visual>
+    <inertial>
+      <origin xyz="0 0 0" rpy="0 0 0" />
+      <mass value="0.01" />
+      <inertia ixx="0.000001" ixy="0.0" ixz="0.0" iyy="0.000001" iyz="0.0" izz="0.000001" />
+    </inertial>
   </link>
   <joint name="camera_optical_joint" type="fixed">

File: src/visionbot_description/description/components/inertia_macros.xacro (robot description, xacro)
@@ -5,7 +5,7 @@
       <xacro:insert_block name="origin" />
       <mass value="${mass}" />
-      <inertia ixx="${(2/5) * mass * (radius*radius)}" ixy="0.0" ixz="0.0"
-        iyy="${(2/5) * mass * (radius*radius)}" iyz="0.0"
-        izz="${(2/5) * mass * (radius*radius)}" />
+      <inertia ixx="${(2.0/5.0) * mass * (radius*radius)}" ixy="0.0" ixz="0.0"
+        iyy="${(2.0/5.0) * mass * (radius*radius)}" iyz="0.0"
+        izz="${(2.0/5.0) * mass * (radius*radius)}" />
     </inertial>
   </xacro:macro>
@@ -14,7 +14,7 @@
       <xacro:insert_block name="origin" />
       <mass value="${mass}" />
-      <inertia ixx="${(1/12) * mass * (y*y+z*z)}" ixy="0.0" ixz="0.0"
-        iyy="${(1/12) * mass * (x*x+z*z)}" iyz="0.0"
-        izz="${(1/12) * mass * (x*x+y*y)}" />
+      <inertia ixx="${(1.0/12.0) * mass * (y*y + z*z)}" ixy="0.0" ixz="0.0"
+        iyy="${(1.0/12.0) * mass * (x*x + z*z)}" iyz="0.0"
+        izz="${(1.0/12.0) * mass * (x*x + y*y)}" />
     </inertial>
   </xacro:macro>
@@ -23,7 +23,7 @@
       <xacro:insert_block name="origin" />
       <mass value="${mass}" />
-      <inertia ixx="${(1/12) * mass * (3*radius*radius + length*length)}" ixy="0.0" ixz="0.0"
-        iyy="${(1/12) * mass * (3*radius*radius + length*length)}" iyz="0.0"
-        izz="${(1/2) * mass * (radius*radius)}" />
+      <inertia ixx="${(1.0/12.0) * mass * (3.0*radius*radius + length*length)}" ixy="0.0" ixz="0.0"
+        iyy="${(1.0/12.0) * mass * (3.0*radius*radius + length*length)}" iyz="0.0"
+        izz="${(0.5) * mass * (radius*radius)}" />
     </inertial>
   </xacro:macro>

File: src/visionbot_description/description/components/lidar.xacro (robot description, xacro)
@@ -13,7 +13,7 @@
     </visual>
     <collision>
-      <origin xyz="0 0 0" rpy="0 0 0" />
+      <origin rpy="0 0 0" xyz="0 0 0" />
       <geometry>
-        <mesh filename="package://visionbot_description/description/meshes/laser_link.stl" />
+        <cylinder length="0.03" radius="0.03" />
       </geometry>
     </collision>

File: src/visionbot_description/description/robot_gazebo.xacro (robot description, xacro)
@@ -2,37 +2,37 @@
 <robot name="robot" xmlns:xacro="http://www.ros.org/wiki/xacro">
   <gazebo reference="rear_left_wheel">
-    <mu1>100000000000000.0</mu1>
-    <mu2>100000000000000.0</mu2>
-    <kp>100000000000000.0</kp>
-    <kd>10.0</kd>
+    <mu1>0.8</mu1>
+    <mu2>0.8</mu2>
+    <kp>1000000.0</kp>
+    <kd>1.0</kd>
     <minDepth>0.001</minDepth>
-    <maxVel>0.1</maxVel>
+    <maxVel>1</maxVel>
     <fdir>1 0 0</fdir>
   </gazebo>
   <gazebo reference="rear_right_wheel">
-    <mu1>100000000000000.0</mu1>
-    <mu2>100000000000000.0</mu2>
-    <kp>100000000000000.0</kp>
-    <kd>10.0</kd>
+    <mu1>0.8</mu1>
+    <mu2>0.8</mu2>
+    <kp>1000000.0</kp>
+    <kd>1.0</kd>
     <minDepth>0.001</minDepth>
-    <maxVel>0.1</maxVel>
+    <maxVel>1</maxVel>
     <fdir>1 0 0</fdir>
   </gazebo>
   <gazebo reference="front_left_wheel">
-    <mu1>100000000000000.0</mu1>
-    <mu2>100000000000000.0</mu2>
-    <kp>100000000000000.0</kp>
-    <kd>10.0</kd>
+    <mu1>0.8</mu1>
+    <mu2>0.8</mu2>
+    <kp>1000000.0</kp>
+    <kd>1.0</kd>
     <minDepth>0.001</minDepth>
-    <maxVel>0.1</maxVel>
+    <maxVel>1</maxVel>
     <fdir>1 0 0</fdir>
   </gazebo>
   <gazebo reference="front_right_wheel">
-    <mu1>100000000000000.0</mu1>
-    <mu2>100000000000000.0</mu2>
-    <kp>100000000000000.0</kp>
-    <kd>10.0</kd>
+    <mu1>0.8</mu1>
+    <mu2>0.8</mu2>
+    <kp>1000000.0</kp>
+    <kd>1.0</kd>
     <minDepth>0.001</minDepth>
-    <maxVel>0.1</maxVel>
+    <maxVel>1</maxVel>
     <fdir>1 0 0</fdir>
   </gazebo>
@@ -70,5 +70,5 @@
   <gazebo>
     <plugin filename="gz_ros2_control-system" name="gz_ros2_control::GazeboSimROS2ControlPlugin">
-      <parameters>/home/gasa14/Workspaces/dev_ws/src/visionbot_launch/config/controllers.yaml</parameters>
+      <parameters>$(find visionbot_control)/config/controllers.yaml</parameters>
     </plugin>
     <plugin filename="gz-sim-sensors-system" name="gz::sim::systems::Sensors">

Commit message: added camera to simulation

File: src/visionbot_description/description/components/camera.xacro (robot description, xacro)
@@ -39,5 +39,5 @@
     <parent link="camera_neck_link" />
     <child link="camera_link" />
-    <origin xyz="0.0075 0 ${camera_offset_z}" rpy="0 ${pi/2} 0" />
+    <origin xyz="0.0075 0 ${camera_offset_z}" rpy="0 0 0" />
   </joint>
   <link name="camera_link">
@@ -61,24 +61,3 @@
   </joint>
   <link name="camera_link_optical"></link>
-  <gazebo reference="camera_link">
-    <sensor name="camera" type="camera">
-      <update_rate>30</update_rate>
-      <topic>camera/image_raw</topic>
-      <camera>
-        <camera_info_topic>camera/camera_info</camera_info_topic>
-        <horizontal_fov>2.09</horizontal_fov>
-        <image>
-          <format>R8G8B8</format>
-          <width>1280</width>
-          <height>720</height>
-        </image>
-        <clip>
-          <near>0.05</near>
-          <far>20.0</far>
-        </clip>
-      </camera>
-      <always_on>true</always_on>
-      <visualize>true</visualize>
-    </sensor>
-  </gazebo>
 </robot>

File: src/visionbot_description/description/robot_gazebo.xacro (robot description, xacro)
@@ -68,13 +68,4 @@
     </sensor>
   </gazebo>
-  <gazebo>
-    <plugin filename="gz_ros2_control-system" name="gz_ros2_control::GazeboSimROS2ControlPlugin">
-      <parameters>$(find visionbot_control)/config/controllers.yaml</parameters>
-    </plugin>
-    <plugin filename="gz-sim-sensors-system" name="gz::sim::systems::Sensors">
-      <render_engine>ogre2</render_engine>
-    </plugin>
-    <plugin filename="gz-sim-imu-system" name="gz::sim::systems::Imu" />
-  </gazebo>
   <gazebo reference="base_link">
     <sensor name="imu" type="imu">
@@ -127,3 +118,37 @@
     </sensor>
   </gazebo>
+  <gazebo reference="camera_link_optical">
+    <sensor name="rpi_camera_module3_wide" type="camera">
+      <always_on>true</always_on>
+      <update_rate>30.0</update_rate>
+      <visualize>true</visualize>
+      <topic>/image_raw</topic>
+      <gz_frame_id>/camera_link_optical</gz_frame_id>
+      <camera name="camera">
+        <horizontal_fov>1.21126</horizontal_fov>
+        <image>
+          <width>2304</width>
+          <height>1296</height>
+          <format>R8G8B8</format>
+        </image>
+        <distortion>
+          <k1>0.0</k1>
+          <k2>0.0</k2>
+          <k3>0.0</k3>
+          <p1>0.0</p1>
+          <p2>0.0</p2>
+          <center>0.5 0.5</center>
+        </distortion>
+      </camera>
+    </sensor>
+  </gazebo>
+  <gazebo>
+    <plugin filename="gz_ros2_control-system" name="gz_ros2_control::GazeboSimROS2ControlPlugin">
+      <parameters>$(find visionbot_control)/config/controllers.yaml</parameters>
+    </plugin>
+    <plugin filename="gz-sim-sensors-system" name="gz::sim::systems::Sensors">
+      <render_engine>ogre2</render_engine>
+    </plugin>
+    <plugin filename="gz-sim-imu-system" name="gz::sim::systems::Imu" />
+  </gazebo>
 </robot>

Commit message: camera topic fix

File: src/visionbot_description/description/components/camera.xacro (robot description, xacro)
@@ -39,5 +39,5 @@
     <parent link="camera_neck_link" />
     <child link="camera_link" />
-    <origin xyz="0.0075 0 ${camera_offset_z}" rpy="0 0 0" />
+    <origin xyz="0.0075 0 ${camera_offset_z}" rpy="0 ${pi/2} 0" />
   </joint>
   <link name="camera_link">
@@ -58,5 +58,5 @@
     <parent link="camera_link" />
     <child link="camera_link_optical" />
-    <origin xyz="0 0 0" rpy="-${pi/2} 0 -${pi/2}" />
+    <origin xyz="0 0 0" rpy="-${pi/2} 0 ${pi/2}" />
   </joint>
   <link name="camera_link_optical"></link>

File: src/visionbot_description/description/robot_gazebo.xacro (robot description, xacro)
@@ -121,9 +121,10 @@
     <sensor name="rpi_camera_module3_wide" type="camera">
       <always_on>true</always_on>
-      <update_rate>30.0</update_rate>
+      <update_rate>20.0</update_rate>
       <visualize>true</visualize>
-      <topic>/image_raw</topic>
-      <gz_frame_id>/camera_link_optical</gz_frame_id>
+      <topic>/camera/image_raw</topic>
       <camera name="camera">
+        <camera_info_topic>/camera/image_raw/camera_info</camera_info_topic>
+        <gz_frame_id>camera_link_optical</gz_frame_id>
         <horizontal_fov>1.21126</horizontal_fov>
         <image>

Commit message: created map by slam for benchmark

File: src/visionbot_description/description/components/camera.xacro (robot description, xacro)
@@ -39,5 +39,5 @@
     <parent link="camera_neck_link" />
     <child link="camera_link" />
-    <origin xyz="0.0075 0 ${camera_offset_z}" rpy="0 ${pi/2} 0" />
+    <origin xyz="0.0075 0 ${camera_offset_z}" rpy="0 ${pi/2.25} 0" />
   </joint>
   <link name="camera_link">
@@ -58,5 +58,5 @@
     <parent link="camera_link" />
     <child link="camera_link_optical" />
-    <origin xyz="0 0 0" rpy="-${pi/2} 0 ${pi/2}" />
+    <origin xyz="0 0 0" rpy="-${pi/2} -${pi/2} ${pi/2}" />
   </joint>
   <link name="camera_link_optical"></link>

File: src/visionbot_description/description/robot_gazebo.xacro (robot description, xacro)
@@ -121,5 +121,5 @@
     <sensor name="rpi_camera_module3_wide" type="camera">
       <always_on>true</always_on>
-      <update_rate>20.0</update_rate>
+      <update_rate>10.0</update_rate>
       <visualize>true</visualize>
       <topic>/camera/image_raw</topic>
@@ -127,8 +127,8 @@
         <camera_info_topic>/camera/image_raw/camera_info</camera_info_topic>
         <gz_frame_id>camera_link_optical</gz_frame_id>
-        <horizontal_fov>1.21126</horizontal_fov>
+        <horizontal_fov>1.78</horizontal_fov>
         <image>
-          <width>2304</width>
-          <height>1296</height>
+          <width>853</width>
+          <height>480</height>
           <format>R8G8B8</format>
         </image>
